File: sound_remocon/sound_remocon.kicad_sch (KiCad schematic)
At the start: 36 parts, among them J1 Conn_01x02_Pin, U1 NJM4580, U2 NJM4580, U3 NJM4580

Commit message: updated
Parts:
- added C1, C2, C3, C4, C5, C6: 0.1u, Capacitor_THT:C_Disc_D3.8mm_W2.6mm_P2.50mm, symbol Device:C
- added Clpf1: C, Capacitor_THT:C_Disc_D3.8mm_W2.6mm_P2.50mm, symbol Device:C
- added R1, R2, R3, R4, R5, R6, Rlpf1, Rmx1, Rmx2, Rmx3, Rna1, Rna2: 10k, Resistor_THT:R_Axial_DIN0207_L6.3mm_D2.5mm_P7.62mm_Horizontal, symbol Device:R
- added Rdiv11, Rdiv12, Rdiv21, Rdiv22, Rdiv31, Rdiv32, Rdiv41, Rdiv42, Rdiv51, Rdiv52, Rdiv61, Rdiv62: R, Resistor_THT:R_Axial_DIN0207_L6.3mm_D2.5mm_P7.62mm_Horizontal, symbol Device:R
- added U4: NJM4580, Package_DIP:DIP-8_W7.62mm, symbol Amplifier_Operational:NJM4580
Connections:
- net +5V: now also Rmx1.1, Rna1.1, U4.8 (V+)
- net GND: now also Clpf1.2, Rdiv12.2, Rdiv22.2, Rdiv32.2, Rdiv42.2, Rdiv52.2, Rdiv62.2, Rmx2.2, Rna2.2, U4.4 (V-)
- net Output_rs: now also Rdiv31.1, Rdiv61.1
- net Output_rx: now also Rdiv11.1, Rdiv41.1
- net Output_ry: now also Rdiv21.1, Rdiv51.1
- new net: Rlpf1.1, Rmx3.1, U4.1
- new net: R1.2, R2.2, R3.2, R4.2, R5.2, R6.2, Rmx3.2, U4.2 (-)
- new net: C3.1, Rdiv31.2, Rdiv32.1
- new net: C3.2, R3.1
- new net: Rmx1.2, Rmx2.1, U4.3 (+)
- new net: C5.1, Rdiv51.2, Rdiv52.1
- new net: C5.2, R5.1
- new net: C2.2, R2.1
- new net: C2.1, Rdiv21.2, Rdiv22.1
- new net: Rna1.2, Rna2.1, U4.5 (+)
- new net: U4.6 (-), U4.7
- new net: C6.1, Rdiv61.2, Rdiv62.1
- new net: C1.1, Rdiv11.2, Rdiv12.1
- new net: C1.2, R1.1
- new net: C6.2, R6.1
- new net: C4.2, R4.1
- new net: C4.1, Rdiv41.2, Rdiv42.1
- new net output: Clpf1.1, Rlpf1.2

Commit message: updated
Parts:
- removed Rdiv11, Rdiv12, Rdiv21, Rdiv22, Rdiv31, Rdiv32, Rdiv41, Rdiv42, Rdiv51, Rdiv52, Rdiv61, Rdiv62: R, Resistor_THT:R_Axial_DIN0207_L6.3mm_D2.5mm_P7.62mm_Horizontal, symbol Device:R
- added Cout1: 4.7u, Capacitor_THT:C_Disc_D4.7mm_W2.5mm_P5.00mm, symbol Device:C
- added J2: Conn_01x02_Pin, Connector_PinHeader_2.54mm:PinHeader_1x02_P2.54mm_Vertical, symbol Connector:Conn_01x02_Pin
- added Rout1, Rout2: 50k, Resistor_THT:R_Axial_DIN0207_L6.3mm_D2.5mm_P7.62mm_Horizontal, symbol Device:R
- Clpf1: value C -> 1n
- Rlpf1: value 10k -> 3.3k
Connections:
- net GND: now also J2.2 (Pin_2), Rout2.2
- net Output_ls: now also C6.1
- net Output_lx: now also C4.1
- net Output_ly: now also C5.1
- net Output_rs: now also C3.1
- net Output_rx: now also C1.1
- net Output_ry: now also C2.1
- net output: now also J2.1 (Pin_1), Rout1.2, Rout2.1; no longer Clpf1.1, Rlpf1.2
- new net: Cout1.2, Rout1.1
- new net: Clpf1.1, Cout1.1, Rlpf1.2

Commit message: updated
Parts:
- added LED1: LED, LED_THT:LED_D3.0mm, symbol Device:LED
- added Rled1: R, Resistor_THT:R_Axial_DIN0207_L6.3mm_D2.5mm_P7.62mm_Horizontal, symbol Device:R
- J2: footprint Connector_PinHeader_2.54mm:PinHeader_1x02_P2.54mm_Vertical -> TerminalBlock:TerminalBlock_bornier-2_P5.08mm
Connections:
- net +5V: now also LED1.2 (A)
- net GND: now also Rled1.2
- new net: LED1.1 (K), Rled1.1
