File: sound_remocon/sound_remocon.kicad_pcb (KiCad board)
At the start: 2 copper layers, 100 x 100 mm, 36 parts, among them J1 Conn_01x02_Pin, U1 NJM4580, U2 NJM4580, U3 NJM4580

Commit message: updated
Parts:
- added C1: 0.1u, Capacitor_THT:C_Disc_D3.8mm_W2.6mm_P2.50mm, F.Cu at (171.5, 63.4)
- added C2: 0.1u, Capacitor_THT:C_Disc_D3.8mm_W2.6mm_P2.50mm, F.Cu at (171.5, 67.5)
- added C3: 0.1u, Capacitor_THT:C_Disc_D3.8mm_W2.6mm_P2.50mm, F.Cu at (171.5, 71.7)
- added C4: 0.1u, Capacitor_THT:C_Disc_D3.8mm_W2.6mm_P2.50mm, F.Cu at (171.5, 75.8)
- added C5: 0.1u, Capacitor_THT:C_Disc_D3.8mm_W2.6mm_P2.50mm, F.Cu at (171.5, 80.0)
- added C6: 0.1u, Capacitor_THT:C_Disc_D3.8mm_W2.6mm_P2.50mm, F.Cu at (177.2, 63.4)
- added Clpf1: C, Capacitor_THT:C_Disc_D3.8mm_W2.6mm_P2.50mm, F.Cu at (177.2, 67.5)
- added R1: 10k, Resistor_THT:R_Axial_DIN0207_L6.3mm_D2.5mm_P7.62mm_Horizontal, F.Cu at (128.4, 29.6)
- added R2: 10k, Resistor_THT:R_Axial_DIN0207_L6.3mm_D2.5mm_P7.62mm_Horizontal, F.Cu at (128.4, 33.7)
- added R3: 10k, Resistor_THT:R_Axial_DIN0207_L6.3mm_D2.5mm_P7.62mm_Horizontal, F.Cu at (128.4, 37.7)
- added R4: 10k, Resistor_THT:R_Axial_DIN0207_L6.3mm_D2.5mm_P7.62mm_Horizontal, F.Cu at (128.4, 41.8)
- added R5: 10k, Resistor_THT:R_Axial_DIN0207_L6.3mm_D2.5mm_P7.62mm_Horizontal, F.Cu at (128.4, 45.8)
- added R6: 10k, Resistor_THT:R_Axial_DIN0207_L6.3mm_D2.5mm_P7.62mm_Horizontal, F.Cu at (128.4, 49.9)
- added Rdiv11: R, Resistor_THT:R_Axial_DIN0207_L6.3mm_D2.5mm_P7.62mm_Horizontal, F.Cu at (128.4, 53.9)
- added Rdiv12: R, Resistor_THT:R_Axial_DIN0207_L6.3mm_D2.5mm_P7.62mm_Horizontal, F.Cu at (128.4, 58.0)
- added Rdiv21: R, Resistor_THT:R_Axial_DIN0207_L6.3mm_D2.5mm_P7.62mm_Horizontal, F.Cu at (128.4, 62.0)
- added Rdiv22: R, Resistor_THT:R_Axial_DIN0207_L6.3mm_D2.5mm_P7.62mm_Horizontal, F.Cu at (128.4, 66.1)
- added Rdiv31: R, Resistor_THT:R_Axial_DIN0207_L6.3mm_D2.5mm_P7.62mm_Horizontal, F.Cu at (128.4, 70.1)
- added Rdiv32: R, Resistor_THT:R_Axial_DIN0207_L6.3mm_D2.5mm_P7.62mm_Horizontal, F.Cu at (128.4, 74.2)
- added Rdiv41: R, Resistor_THT:R_Axial_DIN0207_L6.3mm_D2.5mm_P7.62mm_Horizontal, F.Cu at (128.4, 78.2)
- added Rdiv42: R, Resistor_THT:R_Axial_DIN0207_L6.3mm_D2.5mm_P7.62mm_Horizontal, F.Cu at (139.2, 29.6)
- added Rdiv51: R, Resistor_THT:R_Axial_DIN0207_L6.3mm_D2.5mm_P7.62mm_Horizontal, F.Cu at (139.2, 33.7)
- added Rdiv52: R, Resistor_THT:R_Axial_DIN0207_L6.3mm_D2.5mm_P7.62mm_Horizontal, F.Cu at (139.2, 37.7)
- added Rdiv61: R, Resistor_THT:R_Axial_DIN0207_L6.3mm_D2.5mm_P7.62mm_Horizontal, F.Cu at (139.2, 41.8)
- added Rdiv62: R, Resistor_THT:R_Axial_DIN0207_L6.3mm_D2.5mm_P7.62mm_Horizontal, F.Cu at (139.2, 45.8)
- added Rlpf1: 10k, Resistor_THT:R_Axial_DIN0207_L6.3mm_D2.5mm_P7.62mm_Horizontal, F.Cu at (139.2, 49.9)
- added Rmx1: 10k, Resistor_THT:R_Axial_DIN0207_L6.3mm_D2.5mm_P7.62mm_Horizontal, F.Cu at (150.0, 49.9)
- added Rmx2: 10k, Resistor_THT:R_Axial_DIN0207_L6.3mm_D2.5mm_P7.62mm_Horizontal, F.Cu at (150.0, 53.9)
- added Rmx3: 10k, Resistor_THT:R_Axial_DIN0207_L6.3mm_D2.5mm_P7.62mm_Horizontal, F.Cu at (150.0, 58.0)
- added Rna1: 10k, Resistor_THT:R_Axial_DIN0207_L6.3mm_D2.5mm_P7.62mm_Horizontal, F.Cu at (150.0, 62.0)
- added Rna2: 10k, Resistor_THT:R_Axial_DIN0207_L6.3mm_D2.5mm_P7.62mm_Horizontal, F.Cu at (150.0, 66.1)
- added U4: NJM4580, Package_DIP:DIP-8_W7.62mm, F.Cu at (202.4, -40.0)
- moved J1 158.6 mm to (190.1, 65.8)
- moved Cry1 73.5 mm to (108.0, 53.5)
- moved Crx1 55.7 mm to (90.5, 54.0)
- moved Rly1 51.8 mm to (40.5, 37.4), turned to -90 degrees
- moved JoyStick_right1 50.3 mm to (95.0, 67.4)
- moved Rlx4 49.3 mm to (24.5, 48.8)
- moved Rlx1 48.7 mm to (24.7, 37.4), turned to -90 degrees
- moved U1 48.5 mm to (77.2, 62.9)
- moved Rrx1 45.4 mm to (88.0, 37.4), turned to -90 degrees
- moved Rrx2 44.2 mm to (93.3, 45.0), turned to 90 degrees
- moved Rlx2 42.3 mm to (30.0, 45.0), turned to 90 degrees
- moved Rlx3 41.4 mm to (35.2, 45.0), turned to 90 degrees
- moved Crs1 38.9 mm to (73.0, 53.5)
- moved Rry3 38.3 mm to (114.4, 45.0), turned to 90 degrees
- moved Rly4 34.7 mm to (40.3, 48.8)
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Connections:
- JoyStick_left1 pad a: unconnected-(JoyStick_left1-SWa-Pada) -> Output_l_sw_ac
- JoyStick_left1 pad b: unconnected-(JoyStick_left1-SWb-Padb) -> Output_ls
- JoyStick_left1 pad c: unconnected-(JoyStick_left1-SWc-Padc) -> Output_l_sw_ac
- JoyStick_left1 pad d: unconnected-(JoyStick_left1-SWd-Padd) -> Output_ls
- JoyStick_right1 pad a: unconnected-(JoyStick_right1-SWa-Pada) -> Output_r_sw_ac
- JoyStick_right1 pad b: unconnected-(JoyStick_right1-SWb-Padb) -> Output_rs
- JoyStick_right1 pad c: unconnected-(JoyStick_right1-SWc-Padc) -> Output_r_sw_ac
- JoyStick_right1 pad d: unconnected-(JoyStick_right1-SWd-Padd) -> Output_rs
- Rls3 pad 2: Output_ls -> Output_l_sw_ac
- Rls4 pad 2: Output_ls -> Output_l_sw_ac
- Rrs3 pad 2: Output_rs -> Output_r_sw_ac
- Rrs4 pad 2: Output_rs -> Output_r_sw_ac
- U3 pad 1: Output_ls -> Output_l_sw_ac
- U3 pad 7: Output_rs -> Output_r_sw_ac

Commit message: updated
Parts:
- removed Rdiv11, Rdiv12, Rdiv21, Rdiv22, Rdiv31, Rdiv32, Rdiv41, Rdiv42, Rdiv51, Rdiv52, Rdiv61, Rdiv62: R, Resistor_THT:R_Axial_DIN0207_L6.3mm_D2.5mm_P7.62mm_Horizontal
- added Cout1: 4.7u, Capacitor_THT:C_Disc_D4.7mm_W2.5mm_P5.00mm, F.Cu at (53.6, 44.8)
- added J2: Conn_01x02_Pin, Connector_PinHeader_2.54mm:PinHeader_1x02_P2.54mm_Vertical, F.Cu at (70.7, 34.6)
- added Rout1: 50k, Resistor_THT:R_Axial_DIN0207_L6.3mm_D2.5mm_P7.62mm_Horizontal, F.Cu at (65.6, 47.2)
- added Rout2: 50k, Resistor_THT:R_Axial_DIN0207_L6.3mm_D2.5mm_P7.62mm_Horizontal, F.Cu at (58.6, 39.8)
- Clpf1: value C -> 1n
- Rlpf1: value 10k -> 3.3k
- moved U4 165.5 mm to (64.4, 51.4)
- moved J1 160.8 mm to (31.7, 38.2)
- moved Clpf1 136.0 mm to (44.0, 39.8), turned to -90 degrees
- moved C6 125.0 mm to (52.2, 60.0)
- moved C5 121.6 mm to (52.2, 56.2)
- moved C4 121.6 mm to (52.2, 52.4)
- moved Rlpf1 91.0 mm to (48.2, 47.4), turned to 90 degrees
- moved C3 79.7 mm to (92.6, 60.0), turned to 180 degrees
- moved C2 79.7 mm to (92.6, 56.2), turned to 180 degrees
- moved C1 79.6 mm to (92.6, 52.4), turned to 180 degrees
- moved Rmx1 59.4 mm to (91.4, 39.4), turned to -90 degrees
- moved R6 56.5 mm to (72.0, 47.0), turned to 90 degrees
- moved Rmx2 55.7 mm to (94.7, 47.0), turned to 90 degrees
- moved Rna1 53.8 mm to (101.2, 39.4), turned to -90 degrees
- moved R5 53.2 mm to (75.2, 47.0), turned to 90 degrees
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Connections:
- net output renamed Net-(Clpf1-Pad1)
- C1 pad 1: Net-(C1-Pad1) -> Output_rx
- C2 pad 1: Net-(C2-Pad1) -> Output_ry
- C3 pad 1: Net-(C3-Pad1) -> Output_rs
- C4 pad 1: Net-(C4-Pad1) -> Output_lx
- C5 pad 1: Net-(C5-Pad1) -> Output_ly
- C6 pad 1: Net-(C6-Pad1) -> Output_ls

Commit message: updated
Parts:
- added LED1: LED, LED_THT:LED_D3.0mm, F.Cu at (71.3, 35.0)
- added REF**: 3.2mm_M3, MountingHole:MountingHole_3.2mm_M3, F.Cu at (115.0, 25.0)
- added REF**: 3.2mm_M3, MountingHole:MountingHole_3.2mm_M3, F.Cu at (42.2, 55.0)
- added REF**: 3.2mm_M3, MountingHole:MountingHole_3.2mm_M3, F.Cu at (25.0, 25.0)
- added REF**: 3.2mm_M3, MountingHole:MountingHole_3.2mm_M3, F.Cu at (97.8, 55.0)
- added REF**: 3.2mm_M3, MountingHole:MountingHole_3.2mm_M3, F.Cu at (25.0, 85.0)
- added REF**: 3.2mm_M3, MountingHole:MountingHole_3.2mm_M3, F.Cu at (115.0, 85.0)
- added Rled1: R, Resistor_THT:R_Axial_DIN0207_L6.3mm_D2.5mm_P7.62mm_Horizontal, F.Cu at (73.8, 39.7)
- J1: value Conn_01x02_Pin -> POWER
- J2: value Conn_01x02_Pin -> OUTPUT; footprint Connector_PinHeader_2.54mm:PinHeader_1x02_P2.54mm_Vertical -> TerminalBlock:TerminalBlock_bornier-2_P5.08mm
- JoyStick Left: renamed from JoyStick_left1
- JoyStick Right: renamed from JoyStick_right1
- moved Rmx1 39.9 mm to (82.9, 78.4), turned to 90 degrees
- moved Rna1 39.9 mm to (92.6, 78.4), turned to 90 degrees
- moved Clpf1 36.1 mm to (44.2, 75.9)
- moved JoyStick Left 34.8 mm to (45.0, 37.0)
- moved JoyStick Right 34.8 mm to (95.0, 37.0)
- moved Rout1 32.0 mm to (58.4, 78.4)
- moved Rout2 31.2 mm to (55.0, 70.8)
- moved Rlpf1 31.0 mm to (48.0, 78.4)
- moved Cout1 28.7 mm to (51.6, 73.4), turned to -90 degrees
- moved J1 28.4 mm to (57.9, 27.0)
- moved C6 25.7 mm to (34.2, 78.4)
- moved U2 25.7 mm to (24.2, 70.8)
- moved C4 25.7 mm to (34.2, 70.8)
- moved C5 25.7 mm to (34.2, 74.6)
- moved R1 25.3 mm to (79.6, 70.8), turned to -90 degrees
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Routing:
- net GND: track 0.00 -> 465.0 mm
- net +5V: track 0.00 -> 367.7 mm
- net Output_lx: track 0.00 -> 73.5 mm
- net Output_rx: track 0.00 -> 66.8 mm
- net Net-(Rlpf1-Pad1): track 0.00 -> 61.3 mm
- net Output_ly: track 0.00 -> 59.8 mm
- net output: track 0.00 -> 54.8 mm
- net Output_ry: track 0.00 -> 53.6 mm
- net Net-(U1A-+): track 0.00 -> 45.7 mm
- net Net-(U4A--): track 0.00 -> 45.5 mm
- net Net-(U2A-+): track 0.00 -> 45.2 mm
- net Output_l_sw_ac: track 0.00 -> 44.3 mm
- net Output_rs: track 0.00 -> 43.0 mm
- net Output_r_sw_ac: track 0.00 -> 42.9 mm
- net Output_ls: track 0.00 -> 40.8 mm
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Other:
- board size 100 x 100 mm -> 100 x 70 mm
- board text added: "+5V"
- board text added: "10k"
- board text added: "GND"
- board text added: "Signal"

Commit message: updated
Routing:
- net GND: track 465.0 -> 498.9 mm
- net Net-(C3-Pad2): track 36.1 -> 33.3 mm
- net Output_l_sw_ac: track 44.3 -> 46.5 mm
- net Net-(Rlpf1-Pad1): track 61.3 -> 59.4 mm
- net Net-(C1-Pad2): track 26.0 -> 24.7 mm
- net Net-(U2B--): track 20.3 -> 19.1 mm
- added copper zone on F.Cu, net +5V
- added copper zone on B.Cu, net GND
Other:
- board text added: "Sound Remocon v1.0 MILab 2025 Jan"
