File: kicad/v2/sound_remocon_v2/sound_remocon_v2.kicad_pcb (KiCad board)
At the start: 2 copper layers, 100 x 100 mm, 65 parts, among them SW1 SW_Push, SW2 SW_Push, SW3 SW_Push, SW4 SW_Push, U1 NJM4580

Commit message: updated
Parts:
- R1, R2, R3, R4, Ra1, Ra2, Ra3, Ra4, Ra5, Ra6, Ra7, Ra8, Rb1, Rb2, Rb3, Rb4, Rb5, Rb6, Rb7, Rb8, Rc1, Rc2, Rc3, Rc4, Rc5, Rc6, Rc7, Rc8, Re1, Re2, Rf1, Rg1, Rh1, Rh2, Rled1, Rls1, Rrs1: footprint Resistor_THT:R_Axial_DIN0207_L6.3mm_D2.5mm_P7.62mm_Horizontal -> Resistor_THT:R_Axial_DIN0207_L6.3mm_D2.5mm_P2.54mm_Vertical
- moved Rf1 171.4 mm to (121.5, 118.0)
- moved Rg1 171.4 mm to (121.5, 122.0)
- moved Rh1 171.4 mm to (121.5, 126.1)
- moved Rh2 171.4 mm to (121.5, 130.2)
- moved C10 168.3 mm to (141.0, 115.0)
- moved C9 168.3 mm to (141.0, 110.2)
- moved Re2 162.9 mm to (110.5, 117.0), turned to 180 degrees
- moved Re1 161.0 mm to (108.5, 113.0)
- moved Rc8 156.7 mm to (82.0, 116.0)
- moved Rc7 156.7 mm to (82.0, 111.8)
- moved Rc6 156.6 mm to (82.0, 107.6)
- moved Rc5 156.6 mm to (82.0, 103.4)
- moved Rb3 156.0 mm to (60.9, 95.8)
- moved Rc4 130.5 mm to (82.0, 99.3)
- moved Rc3 130.5 mm to (82.0, 95.1)
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Connections:
- Rb1 pad 1: GND -> Net-(C1-Pad1)
- Rb1 pad 2: Net-(C1-Pad1) -> GND
- Rb2 pad 1: GND -> Net-(C2-Pad1)
- Rb2 pad 2: Net-(C2-Pad1) -> GND
- Rb3 pad 1: GND -> Net-(C3-Pad1)
- Rb3 pad 2: Net-(C3-Pad1) -> GND
- Rb4 pad 1: GND -> Net-(C4-Pad1)
- Rb4 pad 2: Net-(C4-Pad1) -> GND
- Rb5 pad 1: GND -> Net-(C5-Pad1)
- Rb5 pad 2: Net-(C5-Pad1) -> GND
- Rb6 pad 1: GND -> Net-(C6-Pad1)
- Rb6 pad 2: Net-(C6-Pad1) -> GND
- Rb7 pad 1: GND -> Net-(C7-Pad1)
- Rb7 pad 2: Net-(C7-Pad1) -> GND
- Rb8 pad 1: GND -> Net-(C8-Pad1)
- Rb8 pad 2: Net-(C8-Pad1) -> GND
- U1 pad 8: +5V -> Power5V
Other:
- board size 100 x 100 mm -> 100 x 70 mm

Commit message: Updated
Parts:
- added ?: , , F.Cu at (76.2, 62.2)
- added ?: , , F.Cu at (76.2, 52.1)
- added REF**: MountingHole_3.2mm_M3, MountingHole:MountingHole_3.2mm_M3, F.Cu at (146.0, 54.0)
- added REF**: MountingHole_3.2mm_M3, MountingHole:MountingHole_3.2mm_M3, F.Cu at (54.0, 54.0)
- added REF**: MountingHole_3.2mm_M3, MountingHole:MountingHole_3.2mm_M3, F.Cu at (54.0, 116.0)
- added REF**: MountingHole_3.2mm_M3, MountingHole:MountingHole_3.2mm_M3, F.Cu at (146.0, 116.0)
- Rh1: value 50k -> Ro1
- Rh2: value 50k -> Ro2
- moved Ra8 40.4 mm to (84.0, 88.5), turned to -90 degrees
- moved Ra7 34.7 mm to (80.0, 88.5), turned to -90 degrees
- moved Rc1 33.9 mm to (56.0, 108.5), turned to -90 degrees
- moved Rls1 32.0 mm to (114.5, 80.0)
- moved Rg1 32.0 mm to (90.0, 116.5)
- moved Rf1 31.9 mm to (90.0, 113.0)
- moved Rb8 31.2 mm to (84.0, 95.5), turned to -90 degrees
- moved Rrs1 30.6 mm to (114.0, 75.0)
- moved Ra6 29.0 mm to (76.0, 88.5), turned to -90 degrees
- moved C8 28.8 mm to (84.0, 100.5), turned to -90 degrees
- moved Rc2 28.1 mm to (60.0, 108.5), turned to -90 degrees
- moved Rb7 25.9 mm to (80.0, 95.5), turned to -90 degrees
- moved R4 24.2 mm to (142.0, 91.0), turned to 0 degrees
- moved Ra5 23.5 mm to (72.0, 88.5), turned to -90 degrees
- moved C7 22.5 mm to (80.0, 100.5), turned to -90 degrees
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Connections:
- A1 pad 7: SW3 -> SW4
- R4 pad 1: SW3 -> SW4
- Rh1 pad 1: Mixed Signal -> Net-(C10-Pad2)
- Rh1 pad 2: Net-(C10-Pad2) -> Mixed Signal
- Rh2 pad 1: GND -> Mixed Signal
- Rh2 pad 2: Mixed Signal -> GND
- SW4 pad 2: SW3 -> SW4
Routing:
- net Power5V: track 0.00 -> 119.4 mm
Other:
- board text added: "Output Volume = Ro2/(Ro1+Ro2)"

Commit message: updated
Parts:
- Rh1: value Ro1 -> 50k
- Rh2: value Ro2 -> 50k
- moved Power1 68.6 mm to (130.8, 57.1)
- moved ? 48.3 mm to (124.5, 52.1)
- moved ? 48.3 mm to (124.5, 62.2)
- moved SW_PWR1 48.3 mm to (124.5, 54.6)
- moved MixedSignalOut1 39.5 mm to (77.5, 57.1)
- moved Rled1 34.3 mm to (115.6, 59.7)
- moved D1 31.8 mm to (115.6, 54.6), turned to 0 degrees
- moved Rls1 4.92 mm to (115.0, 84.9)
- moved Rrs1 4.91 mm to (115.0, 79.8)
Connections:
- A1 pad 4: SW1 -> SW4
- A1 pad 5: SW2 -> SW3
- A1 pad 6: SW3 -> SW2
- A1 pad 7: SW4 -> SW1
Routing:
- net GND: track 0.00 -> 434.4 mm
- net 3V3: track 0.00 -> 286.0 mm, vias 0 -> 1
- net SW4: track 0.00 -> 81.4 mm
- net Mixed Signal: track 0.00 -> 76.7 mm, vias 0 -> 1
- net SW3: track 0.00 -> 70.4 mm
- net LeftStickSW: track 0.00 -> 67.2 mm
- net LeftStickX: track 0.00 -> 67.2 mm, vias 0 -> 1
- net Net-(U1A--): track 0.00 -> 61.7 mm
- net SW2: track 0.00 -> 60.3 mm
- net LeftStickY: track 0.00 -> 58.8 mm, vias 0 -> 1
- net SW1: track 0.00 -> 58.2 mm
- net Power5V: track 119.4 -> 171.7 mm
- net RightStickY: track 0.00 -> 42.5 mm
- net RightStickSW: track 0.00 -> 42.2 mm
- net Signal1: track 0.00 -> 38.9 mm, vias 0 -> 1
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- added copper zone on F.Cu, net +5V
- added copper zone on F.Cu, net 3V3

Commit message: Updated
Parts:
- Cp2: value 50u -> 47u
- MixedSignalOut1: value Conn_01x02_Pin -> Mixed Signal Out
- Power1: value Conn_01x02_Pin -> Power In
- Rh1: value 50k -> Ro1
- Rh2: value 50k -> Ro2
Routing:
- net Signal8: track 15.3 -> 19.1 mm
- net Signal7: track 18.6 -> 22.0 mm
- net Signal1: track 38.9 -> 41.8 mm
- net Signal6: track 18.1 -> 20.3 mm
- net Mixed Signal: track 76.7 -> 77.7 mm
- net SW2: track 60.3 -> 61.2 mm
- net SW3: track 70.4 -> 71.2 mm
- net SW1: track 58.2 -> 59.0 mm
- net Signal4: track 24.7 -> 25.5 mm, vias 0 -> 1
- net LeftStickY: track 58.8 -> 58.1 mm
- net Signal5: track 21.4 -> 21.9 mm
- net Signal3: track 28.6 -> 28.3 mm, vias 0 -> 1
- net LeftStickSW: vias 0 -> 1
- net Signal2: vias 0 -> 1
- added copper zone on B.Cu, net GND
Other:
- outline, holes or cut-outs redrawn
- board text added: "+5V"
- board text added: "3V3"
- board text added: "GND"
- board text added: "SW"
- board text added: "Signal"
- board text added: "Sound Remocon ver.2 MILab 2025 July"
- board text added: "X"
- board text added: "Y"
- board text added: "nc"
