File: kicad/v2/sound_remocon_v2/sound_remocon_v2.kicad_sch (KiCad schematic)
At the start: 41 parts, among them U1 NJM4580

Commit message: updated
Parts:
- added LeftStick1, RightStick1: RKJXV122400R, myjoystick:RKJXV122400R, symbol joystick:RKJXV122400R
- added LeftStickJ1, LeftStickJ2, RightStickJ1, RightStickJ2: Conn_01x06_Pin, Connector_PinHeader_2.54mm:PinHeader_1x06_P2.54mm_Vertical, symbol Connector:Conn_01x06_Pin
- added R1, R2, R3, R4, R5: 10k, symbol Device:R
- added R35: 50k, symbol Device:R
- added SW1, SW2, SW3: SW_Push, Button_Switch_THT:SW_PUSH_6mm_H7.3mm, symbol Switch:SW_Push
- R34: renamed from R29; value 10k -> 50k
- U1: footprint (none) -> Package_DIP:DIP-8_W7.62mm_Socket
- renumbered R5 to R10, R6 to R11, R7 to R12, R8 to R13, R9 to R14, R10 to R15, R11 to R16, R12 to R17, R13 to R18, R14 to R19, R15 to R20, R16 to R21, R17 to R22, R18 to R23, R19 to R24, R20 to R25, R21 to R26, R22 to R27, R23 to R28, R24 to R29, R25 to R30, R26 to R31, R27 to R32, R28 to R33, R1 to R6, R2 to R7, R3 to R8, R4 to R9
Connections:
- net GND: now also LeftStick1.3 (Rx3), LeftStick1.4 (Ry1), LeftStickJ1.1 (Pin_1), LeftStickJ2.1 (Pin_1), R1.2, R2.2, R3.2, R35.1, R4.2, R5.2, RightStick1.3 (Rx3), RightStick1.4 (Ry1), RightStickJ1.1 (Pin_1), RightStickJ2.1 (Pin_1); no longer R34.1
- net Mixed Signal: now also R34.1, R35.2; no longer C10.2, R34.2
- net LeftStickSW: now reaches A1.27 (GPIO21)
- net LeftStickSW: now also LeftStick1.b (SWb), LeftStick1.d (SWd), LeftStickJ1.6 (Pin_6), LeftStickJ2.6 (Pin_6), R1.1
- net RightStickSW: now reaches A1.29 (GPIO22)
- net RightStickSW: now also R2.1, RightStick1.b (SWb), RightStick1.d (SWd), RightStickJ1.6 (Pin_6), RightStickJ2.6 (Pin_6)
- net LeftStickX: now reaches A1.31 (GPIO26_ADC0)
- net LeftStickX: now also LeftStick1.2 (Rx2), LeftStickJ1.3 (Pin_3), LeftStickJ2.3 (Pin_3)
- net LeftStickY: now reaches A1.32 (GPIO27_ADC1)
- net LeftStickY: now also LeftStick1.5 (Ry2), LeftStickJ1.4 (Pin_4), LeftStickJ2.4 (Pin_4)
- net RightStickY: now reaches A1.34 (GPIO28_ADC2)
- net RightStickY: now also RightStick1.5 (Ry2), RightStickJ1.4 (Pin_4), RightStickJ2.4 (Pin_4)
- net 3V3: now reaches A1.36 (3V3)
- net 3V3: now also LeftStick1.1 (Rx1), LeftStick1.6 (Ry3), LeftStick1.a (SWa), LeftStick1.c (SWc), LeftStickJ1.2 (Pin_2), LeftStickJ1.5 (Pin_5), LeftStickJ2.2 (Pin_2), LeftStickJ2.5 (Pin_5), RightStick1.1 (Rx1), RightStick1.6 (Ry3), RightStick1.a (SWa), RightStick1.c (SWc), RightStickJ1.2 (Pin_2), RightStickJ1.5 (Pin_5), RightStickJ2.2 (Pin_2), RightStickJ2.5 (Pin_5), SW1.1, SW2.1, SW3.1
- net SW1: now reaches A1.4 (GPIO2)
- net SW1: now also R3.1, SW1.2
- net SW2: now reaches A1.5 (GPIO3)
- net SW2: now also R4.1, SW2.2
- net SW3: now reaches A1.6 (GPIO4)
- net SW3: now also R5.1, SW3.2
- new net: RightStickJ1.3 (Pin_3), RightStickJ2.3 (Pin_3)
- new net: C10.2, R34.2
- no-connect marks 0 -> 16
Other:
- moved on the sheet: A1, C1, C10, C2, C3, C4, C5, C6, C7, C8, C9, R10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

Commit message: updated
Parts:
- added Cp1: 0.1u, Capacitor_THT:C_Disc_D5.1mm_W3.2mm_P5.00mm, symbol Device:C
- added Cp2: 50u, Capacitor_THT:CP_Radial_D8.0mm_P5.00mm, symbol Device:C_Polarized
- added MixedSignalOut1, Power1: Conn_01x02_Pin, TerminalBlock:TerminalBlock_bornier-2_P5.08mm, symbol Connector:Conn_01x02_Pin
- added SW1: SW_SPDT, Connector_PinHeader_2.54mm:PinHeader_1x03_P2.54mm_Vertical, symbol Switch:SW_SPDT
- C1, C2, C3, C4, C5, C6, C7, C8: footprint (none) -> Capacitor_THT:C_Disc_D5.1mm_W3.2mm_P5.00mm
- C10: value C -> 4.7u; footprint (none) -> Capacitor_THT:C_Disc_D5.1mm_W3.2mm_P5.00mm
- C9: value C -> 1000p; footprint (none) -> Capacitor_THT:C_Disc_D5.1mm_W3.2mm_P5.00mm
- R1: renamed from R3; footprint (none) -> Resistor_THT:R_Axial_DIN0207_L6.3mm_D2.5mm_P7.62mm_Horizontal
- R2: renamed from R4; footprint (none) -> Resistor_THT:R_Axial_DIN0207_L6.3mm_D2.5mm_P7.62mm_Horizontal
- R3: renamed from R5; footprint (none) -> Resistor_THT:R_Axial_DIN0207_L6.3mm_D2.5mm_P7.62mm_Horizontal
- R4: renamed from R16; footprint (none) -> Resistor_THT:R_Axial_DIN0207_L6.3mm_D2.5mm_P7.62mm_Horizontal
- R5: renamed from R26; footprint (none) -> Resistor_THT:R_Axial_DIN0207_L6.3mm_D2.5mm_P7.62mm_Horizontal
- R6: renamed from R27; footprint (none) -> Resistor_THT:R_Axial_DIN0207_L6.3mm_D2.5mm_P7.62mm_Horizontal
- R7: renamed from R28; footprint (none) -> Resistor_THT:R_Axial_DIN0207_L6.3mm_D2.5mm_P7.62mm_Horizontal
- R8: renamed from R29; footprint (none) -> Resistor_THT:R_Axial_DIN0207_L6.3mm_D2.5mm_P7.62mm_Horizontal
- Ra1: renamed from R6; footprint (none) -> Resistor_THT:R_Axial_DIN0207_L6.3mm_D2.5mm_P7.62mm_Horizontal
- Ra2: renamed from R7; footprint (none) -> Resistor_THT:R_Axial_DIN0207_L6.3mm_D2.5mm_P7.62mm_Horizontal
- Ra3: renamed from R8; footprint (none) -> Resistor_THT:R_Axial_DIN0207_L6.3mm_D2.5mm_P7.62mm_Horizontal
- Ra4: renamed from R9; footprint (none) -> Resistor_THT:R_Axial_DIN0207_L6.3mm_D2.5mm_P7.62mm_Horizontal
- Ra5: renamed from R10; footprint (none) -> Resistor_THT:R_Axial_DIN0207_L6.3mm_D2.5mm_P7.62mm_Horizontal
- Ra6: renamed from R11; footprint (none) -> Resistor_THT:R_Axial_DIN0207_L6.3mm_D2.5mm_P7.62mm_Horizontal
- Ra7: renamed from R12; footprint (none) -> Resistor_THT:R_Axial_DIN0207_L6.3mm_D2.5mm_P7.62mm_Horizontal
- Ra8: renamed from R13; footprint (none) -> Resistor_THT:R_Axial_DIN0207_L6.3mm_D2.5mm_P7.62mm_Horizontal
- Rb1: renamed from R14; footprint (none) -> Resistor_THT:R_Axial_DIN0207_L6.3mm_D2.5mm_P7.62mm_Horizontal
- Rb2: renamed from R15; footprint (none) -> Resistor_THT:R_Axial_DIN0207_L6.3mm_D2.5mm_P7.62mm_Horizontal
- Rb3: renamed from R17; footprint (none) -> Resistor_THT:R_Axial_DIN0207_L6.3mm_D2.5mm_P7.62mm_Horizontal
- Rb4: renamed from R18; footprint (none) -> Resistor_THT:R_Axial_DIN0207_L6.3mm_D2.5mm_P7.62mm_Horizontal
- Rb5: renamed from R19; footprint (none) -> Resistor_THT:R_Axial_DIN0207_L6.3mm_D2.5mm_P7.62mm_Horizontal
- Rb6: renamed from R20; footprint (none) -> Resistor_THT:R_Axial_DIN0207_L6.3mm_D2.5mm_P7.62mm_Horizontal
- Rb7: renamed from R21; footprint (none) -> Resistor_THT:R_Axial_DIN0207_L6.3mm_D2.5mm_P7.62mm_Horizontal
- Rc1: renamed from R22; footprint (none) -> Resistor_THT:R_Axial_DIN0207_L6.3mm_D2.5mm_P7.62mm_Horizontal
- Rc2: renamed from R23; footprint (none) -> Resistor_THT:R_Axial_DIN0207_L6.3mm_D2.5mm_P7.62mm_Horizontal
- Rc3: renamed from R24; footprint (none) -> Resistor_THT:R_Axial_DIN0207_L6.3mm_D2.5mm_P7.62mm_Horizontal
- Rc4: renamed from R25; footprint (none) -> Resistor_THT:R_Axial_DIN0207_L6.3mm_D2.5mm_P7.62mm_Horizontal
- Re1: renamed from R30; footprint (none) -> Resistor_THT:R_Axial_DIN0207_L6.3mm_D2.5mm_P7.62mm_Horizontal
- Re2: renamed from R31; footprint (none) -> Resistor_THT:R_Axial_DIN0207_L6.3mm_D2.5mm_P7.62mm_Horizontal
- Rf1: renamed from R32; footprint (none) -> Resistor_THT:R_Axial_DIN0207_L6.3mm_D2.5mm_P7.62mm_Horizontal
- Rg1: renamed from R33; footprint (none) -> Resistor_THT:R_Axial_DIN0207_L6.3mm_D2.5mm_P7.62mm_Horizontal
- Rh1: renamed from R34; footprint (none) -> Resistor_THT:R_Axial_DIN0207_L6.3mm_D2.5mm_P7.62mm_Horizontal
- Rh2: renamed from R35; footprint (none) -> Resistor_THT:R_Axial_DIN0207_L6.3mm_D2.5mm_P7.62mm_Horizontal
- Rls1: renamed from R1; footprint (none) -> Resistor_THT:R_Axial_DIN0207_L6.3mm_D2.5mm_P7.62mm_Horizontal
- Rrs1: renamed from R2; footprint (none) -> Resistor_THT:R_Axial_DIN0207_L6.3mm_D2.5mm_P7.62mm_Horizontal
- renumbered SW1 to SW2, SW2 to SW3, SW3 to SW4
Connections:
- net +5V: now also Power1.2 (Pin_2), SW1.2 (B); no longer A1.39 (VSYS), Re1.1
- net GND: now also Cp1.2, Cp2.2, MixedSignalOut1.1 (Pin_1), Power1.1 (Pin_1)
- net Mixed Signal: now also MixedSignalOut1.2 (Pin_2)
- new net Power5V: A1.39 (VSYS), Cp1.1, Cp2.1, Re1.1, SW1.1 (A)
- no-connect marks 16 -> 17
Other:
- moved on the sheet: U1B, U1C

Commit message: updated
Parts:
- added D1: LED, LED_THT:LED_D3.0mm, symbol Device:LED
- added R4: 10k, Resistor_THT:R_Axial_DIN0207_L6.3mm_D2.5mm_P7.62mm_Horizontal, symbol Device:R
- added Rled1: 1k, Resistor_THT:R_Axial_DIN0207_L6.3mm_D2.5mm_P7.62mm_Horizontal, symbol Device:R
- added SW4: SW_Push, Button_Switch_THT:SW_PUSH_6mm_H7.3mm, symbol Switch:SW_Push
- renumbered R4 to Rb3, Rb3 to Rb4, Rb4 to Rb5, Rb5 to Rb6, Rb6 to Rb7, Rb7 to Rb8, R5 to Rc5, R6 to Rc6, R7 to Rc7, R8 to Rc8, SW2 to SW1, SW3 to SW2, SW4 to SW3, SW1 to SW_PWR1
Connections:
- net 3V3: now also SW4.1
- net GND: now also R4.2, Rled1.2
- net Power5V: now also D1.2 (A)
- net SW3: now also A1.7 (GPIO5), R4.1, SW4.2
- new net: D1.1 (K), Rled1.1
- no-connect marks 17 -> 16

Commit message: updated
Parts:
- R1, R2, R3, R4, Ra1, Ra2, Ra3, Ra4, Ra5, Ra6, Ra7, Ra8, Rb1, Rb2, Rb3, Rb4, Rb5, Rb6, Rb7, Rb8, Rc1, Rc2, Rc3, Rc4, Rc5, Rc6, Rc7, Rc8, Re1, Re2, Rf1, Rg1, Rh1, Rh2, Rled1, Rls1, Rrs1: footprint Resistor_THT:R_Axial_DIN0207_L6.3mm_D2.5mm_P7.62mm_Horizontal -> Resistor_THT:R_Axial_DIN0207_L6.3mm_D2.5mm_P2.54mm_Vertical
Connections:
- net +5V: no longer U1.8 (V+)
- net GND: now also Rb1.2, Rb2.2, Rb3.2, Rb4.2, Rb5.2, Rb6.2, Rb7.2, Rb8.2; no longer Rb1.1, Rb2.1, Rb3.1, Rb4.1, Rb5.1, Rb6.1, Rb7.1, Rb8.1
- net Power5V: now also U1.8 (V+)
- net at C5.1, Ra5.2: now also Rb5.1; no longer Rb5.2
- net at C3.1, Ra3.2: now also Rb3.1; no longer Rb3.2
- net at C2.1, Ra2.2: now also Rb2.1; no longer Rb2.2
- net at C1.1, Ra1.2: now also Rb1.1; no longer Rb1.2
- net at C6.1, Ra6.2: now also Rb6.1; no longer Rb6.2
- net at C7.1, Ra7.2: now also Rb7.1; no longer Rb7.2
- net at C8.1, Ra8.2: now also Rb8.1; no longer Rb8.2
- net at C4.1, Ra4.2: now also Rb4.1; no longer Rb4.2
Other:
- moved on the sheet: Rb1, Rb2, Rb3, Rb4, Rb5, Rb6, Rb7, Rb8

Commit message: Updated
Connections:
- net GND: now also Rh2.2; no longer Rh2.1
- net Mixed Signal: now also Rh1.2, Rh2.1; no longer Rh1.1, Rh2.2
- net SW3: no longer A1.7 (GPIO5), R4.1, SW4.2
- net at C10.2: now also Rh1.1; no longer Rh1.2
- new net SW4: A1.7 (GPIO5), R4.1, SW4.2
Other:
- moved on the sheet: Rh1, Rh2
Changed lines of the file:
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@@
 	)
 	(junction
+		(at 363.22 111.76)
+		(diameter 0)
+		(color 0 0 0 0)
+	)
+	(junction
 		(at 59.69 199.39)
 		(diameter 0)
@@
 	)
 	(junction
-		(at 363.22 111.76)
-		(diameter 0)
-		(color 0 0 0 0)
-	)
-	(junction
 		(at 26.67 24.13)
 		(diameter 0)
@@
 		)
 	)
-	(global_label "SW3"
+	(global_label "SW4"
 		(shape input)
 		(at 58.42 80.01 180)
@@
 		)
 	)
-	(global_label "SW3"
+	(global_label "SW4"
 		(shape input)
 		(at 215.9 186.69 0)
@@
 	(symbol
 		(lib_id "Device:R")
-		(at 363.22 107.95 180)
+		(at 363.22 107.95 0)
 		(unit 1)
 		(exclude_from_sim no)
@@
 		(dnp no)
 		(property "Reference" "Rh1"
-			(at 360.934 107.95 90)
+			(at 365.506 107.95 90)
 			(effects
 				(font
@@
 		)
 		(property "Value" "50k"
-			(at 365.76 107.95 90)
+			(at 360.68 107.95 90)
 			(effects
 				(font
@@
 		)
 		(property "Footprint" "Resistor_THT:R_Axial_DIN0207_L6.3mm_D2.5mm_P2.54mm_Vertical"
-			(at 364.998 107.95 90)
+			(at 361.442 107.95 90)
 			(effects
 				(font
@@
 	(symbol
 		(lib_id "Device:R")
-		(at 363.22 115.57 180)
+		(at 363.22 115.57 0)
 		(unit 1)
 		(exclude_from_sim no)
@@
 		(dnp no)
 		(property "Reference" "Rh2"
-			(at 360.934 115.57 90)
+			(at 365.506 115.57 90)
 			(effects
 				(font
@@
 		)
 		(property "Value" "50k"
-			(at 365.76 115.57 90)
+			(at 360.68 115.57 90)
 			(effects
 				(font
@@
 		)
 		(property "Footprint" "Resistor_THT:R_Axial_DIN0207_L6.3mm_D2.5mm_P2.54mm_Vertical"
-			(at 364.998 115.57 90)
+			(at 361.442 115.57 90)
 			(effects
 				(font

Commit message: updated
Connections:
- net SW1: now also A1.7 (GPIO5); no longer A1.4 (GPIO2)
- net SW2: now also A1.6 (GPIO4); no longer A1.5 (GPIO3)
- net SW3: now also A1.5 (GPIO3); no longer A1.6 (GPIO4)
- net SW4: now also A1.4 (GPIO2); no longer A1.7 (GPIO5)
Changed lines of the file:
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@@
 		)
 	)
-	(global_label "SW3"
+	(global_label "SW2"
 		(shape input)
 		(at 58.42 77.47 180)
@@
 		)
 	)
-	(global_label "SW4"
+	(global_label "SW1"
 		(shape input)
 		(at 58.42 80.01 180)
@@
 		)
 	)
-	(global_label "SW1"
+	(global_label "SW4"
 		(shape input)
 		(at 58.42 72.39 180)
@@
 		)
 	)
-	(global_label "SW2"
+	(global_label "SW3"
 		(shape input)
 		(at 58.42 74.93 180)

Commit message: Updated
Parts:
- Cp2: value 50u -> 47u
Changed lines of the file:
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@@
 			)
 		)
-		(property "Value" "50u"
+		(property "Value" "47u"
 			(at 389.89 62.6109 0)
 			(effects
